Commit message: add safety sensors

File: e100_description/include/urdf/ria_e100_gazebo.urdf.xacro (robot description, xacro)
@@ -1,4 +1,5 @@
 <?xml version="1.0"?>
 <robot name="ria_e100_gazebo" xmlns:xacro="http://www.ros.org/wiki/xacro">
+  <xacro:arg name="safety_sensors_enabled" default="$(optenv SAFETY_SENSORS_ENABLED)"/>
   <xacro:include filename="$(find e100_description)/include/urdf/ria_e100_gazebo_core.urdf.xacro"/>
   <xacro:ria_e100 base_hw_interface="hardware_interface/VelocityJointInterface"/>

File: e100_description/include/urdf/ria_e100_gazebo_core.urdf.xacro (robot description, xacro)
@@ -1,4 +1,5 @@
 <?xml version="1.0"?>
 <robot name="RIA-E100" xmlns:xacro="http://www.ros.org/wiki/xacro">
+  <xacro:arg name="safety_sensors_enabled" default="false" />
   <xacro:include filename="$(find e100_description)/include/urdf/materials.urdf.xacro"/>
   <xacro:include filename="$(find e100_description)/include/urdf/property.urdf.xacro"/>
@@ -7,4 +8,7 @@
   <xacro:include filename="$(find e100_description)/include/urdf/rgbd.urdf.xacro"/>
   <xacro:include filename="$(find e100_description)/include/urdf/imu.urdf.xacro"/>
+  <xacro:if value="$(arg safety_sensors_enabled)">
+   <xacro:include filename="$(find e100_description)/include/urdf/safety_sensors.urdf.xacro"/>
+  </xacro:if>
   <xacro:macro name="ria_e100" params="base_hw_interface:=hardware_interface/VelocityJointInterface">
   <link name="base_link">
@@ -164,4 +168,4 @@
     <turnGravityOff>false</turnGravityOff>
   </gazebo>
-  </xacro:macro>
+ </xacro:macro>
 </robot>
